Commit message: working version for ROS kinetic@

File: single_lwr_example/single_lwr_robot/robot/single_lwr_robot.urdf.xacro (robot description, xacro)
@@ -3,5 +3,5 @@
 	<!-- Include all models -->
 	<xacro:include filename="$(find lwr_description)/model/kuka_lwr.urdf.xacro"/>
-	<!-- and assemble your robot -->
+	<!-- and assemble your robot
 	<link name="box">
 		<inertial>
@@ -28,7 +28,7 @@
 	<gazebo reference="box">
 		<static>true</static>>
-	</gazebo>
+	</gazebo> -->
 	<!-- using the models -->
-	<xacro:kuka_lwr parent="box" name="lwr">
+	<xacro:kuka_lwr name="lwr">
 		<origin xyz="0 0 1" rpy="0 0 0"/>
 	</xacro:kuka_lwr>
