Commit message: updates for boris integration, everything still works

File: lwr_description/model/kuka_lwr.urdf.xacro (robot description, xacro)
@@ -20,15 +20,15 @@
   <xacro:property name="rate_daming" value="20000"/>
   <!-- URDF model with default base_link (world)-->
-  <xacro:macro name="kuka_lwr" params="name base_link:=world *origin">
-    <link name="${base_link}"/>
-    <gazebo reference="${base_link}">
+  <xacro:macro name="kuka_lwr" params="parent name *origin">
+    <!-- <link name="${base_link}"/> -->
+    <!-- <gazebo reference="${base_link}">
       <static>true</static>
       <turnGravityOff>true</turnGravityOff>
-    </gazebo>
+    </gazebo> -->
     <!-- First (shoulder) element of the arm. Fixed to its parent. -->
     <joint name="${name}_base_joint" type="fixed">
       <xacro:insert_block name="origin"/>
       <origin xyz="0 0 0" rpy="0 0 0"/>
-      <parent link="${base_link}"/>
+      <parent link="${parent}"/>
       <child link="${name}_base_link"/>
     </joint>

File: single_lwr_example/single_lwr_robot/robot/single_lwr_robot.urdf.xacro (robot description, xacro)
@@ -29,6 +29,7 @@
 		<static>true</static>>
 	</gazebo> -->
+	<link name="world" />
 	<!-- using the models -->
-	<xacro:kuka_lwr name="lwr">
+	<xacro:kuka_lwr name="lwr" parent="world">
 		<origin xyz="0 0.12853 0.20722" rpy="0 ${-75 * M_PI / 180} ${-90 * M_PI / 180}"/>
 	</xacro:kuka_lwr>
